File: C64 JoyAdapter/C64 JoyAdapter.kicad_pcb (KiCad board)
At the start: 2 copper layers, 82.5 x 40.6 mm, 13 parts, among them J1 Port 1, J2 Port 2, M1 Mounting, M2 Mounting, M3 Mounting, M4 Mounting, M5 Mounting, M6 Mounting

Commit message: Layout done
Parts:
- removed M5, M6: Mounting, mounting:M3_pin
- added A1: Arduino_Pro_Micro, arduino_pro_micro:Arduino_Pro_Micro, F.Cu at (159.4, 92.1)
- added D1: PWR, LED_THT:LED_D5.0mm_Clear, F.Cu at (163.2, 108.6)
- added J3: C64 JoyKEY, C64_IDC:IDC_Joystick, F.Cu at (99.7, 87.0)
- added SW1: RESET, Button_Switch_THT:SW_Tactile_SPST_Angled_PTS645Vx39-2LFS, F.Cu at (161.9, 74.3)
- added SW2: MODE, Button_Switch_THT:SW_Tactile_SPST_Angled_PTS645Vx39-2LFS, F.Cu at (150.5, 74.3)
- moved R4 85.8 mm to (133.3, 90.2), turned to 180 degrees
- moved R5 72.0 mm to (133.3, 94.0), turned to 180 degrees
- moved R2 60.6 mm to (108.6, 92.1)
- moved R1 60.6 mm to (108.6, 88.3)
- moved R3 47.4 mm to (108.6, 95.9)
- moved J1 29.6 mm to (128.9, 82.7), turned to 180 degrees
- moved M2 3.81 mm to (173.4, 75.6)
- moved M4 3.81 mm to (173.4, 108.6)
- moved M1 2.54 mm to (99.7, 108.6)
- moved M3 2.54 mm to (99.7, 75.6)
- moved J2 0.95 mm to (117.8, 101.5)
Routing:
- net VCC: track 0.00 -> 154.0 mm, vias 0 -> 2
- net GND: track 133.2 -> 0.00 mm
- net POT_BY: track 0.00 -> 101.2 mm, vias 0 -> 2
- net P2_UP: track 9.90 -> 84.2 mm
- net P2_DOWN: track 13.2 -> 83.6 mm, vias 0 -> 3
- net P2_RIGHT: track 14.0 -> 75.6 mm, vias 0 -> 1
- net P2_LEFT: track 13.8 -> 72.4 mm, vias 0 -> 3
- net P2_FIRE: track 14.2 -> 72.3 mm, vias 0 -> 2
- net POT_AY: track 0.00 -> 57.5 mm, vias 0 -> 4
- net POT_BX: track 18.6 -> 73.9 mm, vias 0 -> 4
- net P1_FIRE: track 15.5 -> 70.5 mm
- net /FIRE1: track 54.8 -> 0.00 mm
- net /UP: track 52.7 -> 0.00 mm, vias 1 -> 0
- net /FIRE2: track 52.1 -> 0.00 mm, vias 1 -> 0
- net /DOWN: track 45.8 -> 0.00 mm, vias 1 -> 0
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- added copper zone on B.Cu, net GND
Other:
- board size 82.5 x 40.6 mm -> 81.3 x 40.6 mm
- board text added: "C64 JoyKEY"
- board text added: "Commodore 64 Joystick Adapter"
- board text added: "MODE"
- board text added: "PORT 1"
- board text added: "PORT 2"
- board text added: "RESET"
- board text added: "SYS"
- board text removed: "6x 1n4148"
- board text removed: "Amstrad CPC464 Joystick Splitter"
- board text removed: "JOYSTICK 0"
- board text removed: "JOYSTICK 1"
