File: C64 JoyAdapter/C64 JoyAdapter.sch (KiCad schematic (older format))
At the start: 17 parts, among them J1 Port 1, J2 Port 2, M1 Mounting, M2 Mounting, M3 Mounting, M4 Mounting, M5 Mounting, M6 Mounting, SW1 RESET, SW2 MODE

Commit message: Layout done
Parts:
- removed M5, M6: Mounting, mounting:M3_pin, symbol mounting:Mounting
- added J3: C64 JoyKEY, C64_IDC:IDC_Joystick, symbol c64_idc:C64_IDC2_OUT
- A1: symbol promicro:Arduino_Pro_Micro -> arduino_pro_micro:Arduino_Pro_Micro
- D1: footprint LEDs:LED_D5.0mm -> LED_THT:LED_D5.0mm_Clear
- SW1, SW2: footprint Buttons_Switches_THT:SW_PUSH_6mm -> Button_Switch_THT:SW_Tactile_SPST_Angled_PTS645Vx39-2LFS
Connections:
- net GND: now also J3.8 (Pin_8)
- net P2_DOWN: now also J3.2 (Pin_2)
- net P2_FIRE: now also J3.6 (Pin_6)
- net P2_LEFT: now also J3.3 (Pin_3)
- net P2_RIGHT: now also J3.4 (Pin_4)
- net P2_UP: now also J3.1 (Pin_1)
- net POT_BX: now also J3.9 (Pin_9)
- net POT_BY: now also J3.5 (Pin_5)
- net VCC: now also J3.7 (Pin_7)
Other:
- moved on the sheet: J1, J2, R1, R2, R3, R4
